File: BEP2022_PCB/Gen3/untitled.brd (EAGLE design)
At the start: 10 parts, among them U1 MCP2562-E/P, X1 JST-XH-03-PIN-LONG-PAD, X2 JST-XH-04-PIN-LONG-PAD, X3 JST-XH-04-PIN-LONG-PAD, X4 JST-XH-03-PIN-LONG-PAD

Commit message: update PCB
Parts:
- added C1, C2, C3: 4.7uF, SparkFun-Capacitors:0603
- added C4, C5: 0.1uF, SparkFun-Capacitors:0603
- added R2: 10K, SparkFun-Resistors:0603
- added R4, R5: 100K, SparkFun-Resistors:0603
- added U2: ESP32-WROOM-32E_(16MB), ESP32-WROOM-32E__16MB_:XCVR_ESP32-WROOM-32E_(16MB)
- added U3: NJM2845DL1-33-TE1, NJM2845DL1-33-TE1:DPAK228P968X238-4N
- U$1: value ESP32DEVKITV1 -> 2N7002DW; device ESP32-DEVKITV1:ESP32-DEVKITV1 -> 2N7002DW:SOT363
- moved U$1 54.6 mm to (-20.8, -14.1)
Connections:
- new net DTR: R4.2, U$1.2, U$1.4
- new net EN: C1.1, U$1.6, U2.3
- new net IO0: R2.1, U$1.3, U2.25
- new net LED: U2.24
- new net N$3: R4.1, R5.1
- new net RTS: R5.2, U$1.1, U$1.5
- new net RXD0: U2.34
- new net SCL: U2.36
- new net SDA: U2.33
- new net TXD0: U2.35
- new net VIN: C3.2, C4.1, U3.1
- net 1WIRE: now also U2.9; no longer U$1.D33
- net 3V3: now also C2.1, C5.2, R2.2, U2.2, U3.3; no longer U$1.3V3
- net AIN: now also U2.8; no longer U$1.D32
- net CAN_RX: no longer U$1.D25
- net CAN_TX: no longer U$1.D26
- net GND: now also C1.2, C2.2, C3.1, C4.2, C5.1, U2.1, U2.15, U2.38, U2.39_1, U2.39_2, U2.39_3, U2.39_4, U2.39_5, U2.39_6, U2.39_7, U2.39_8, U2.39_9, U3.2; no longer U$1.GND@1, U$1.GND@2
- net VDD_5V: no longer U$1.VIN
Routing:
- net GND: track 122.8 -> 0.00 mm, vias 2 -> 0
- net VDD_5V: track 107.3 -> 0.00 mm
- net CANL: track 90.6 -> 0.00 mm
- net CANH: track 83.5 -> 0.00 mm
- net 3V3: track 48.5 -> 0.00 mm, vias 1 -> 0
- net AIN: track 34.5 -> 0.00 mm, vias 2 -> 0
- net 1WIRE: track 33.0 -> 0.00 mm, vias 1 -> 0
- net CAN_RX_5V: track 23.1 -> 0.00 mm
- net CAN_TX_5V: track 16.7 -> 0.00 mm
- net CAN_TX: track 3.77 -> 0.00 mm
- net CAN_RX: track 3.77 -> 0.00 mm
