File: BEP2022_PCB/Gen3/untitled.sch (EAGLE design)
At the start: 17 parts, among them U1 MCP2562-E/P, X1 JST-XH-03-PIN-LONG-PAD, X2 JST-XH-04-PIN-LONG-PAD, X3 JST-XH-04-PIN-LONG-PAD, X4 JST-XH-03-PIN-LONG-PAD

Commit message: update PCB
Parts:
- removed R3: 1k, SparkFun-Resistors:1KOHM-0603-1/10W-1%
- removed U$3: (no value), AE-BNO055:AE-BNO055-BO
- added C5: 0.1uF, SparkFun-Capacitors:0.1UF-0603-25V-(+80/-20%)
- added R5: 100K, SparkFun-Resistors:4.7KOHM-0603-1/10W-1%
- added U$2: BAT, BAT:BAT
- added U2: ESP32-WROOM-32E_(16MB), ESP32-WROOM-32E__16MB_:ESP32-WROOM-32E_(16MB)
- added U3: NJM2845DL1-33-TE1, NJM2845DL1-33-TE1:NJM2845DL1-33-TE1
- C4: value 4.7uF -> 0.1uF; device SparkFun-Capacitors:4.7UF-0603-6.3V-(10%) -> SparkFun-Capacitors:0.1UF-0603-25V-(+80/-20%)
- R2: value 1k -> 10K; device SparkFun-Resistors:1KOHM-0603-1/10W-1% -> SparkFun-Resistors:4.7KOHM-0603-1/10W-1%
- R4: value 4.7k -> 100K
- U$1: value ESP32DEVKITV1 -> 2N7002DW; device ESP32-DEVKITV1:ESP32DEVKITV1 -> 2N7002DW:2N7002DW
Connections:
- new net DTR: R4.2, U$1.G1, U$1.S2
- new net IO0: R2.1, U$1.D2, U2.IO0
- new net LED: U2.IO2
- new net N$3: R4.1, R5.1
- new net RTS: R5.2, U$1.G2, U$1.S1
- new net RXD0: U2.RXD0
- new net TXD0: U2.TXD0
- new net VIN: C3.2, C4.1, U3.VIN
- net 1WIRE: now also U2.IO33; no longer R4.1, U$1.IO33
- net 3V3: now also C5.2, U2.3V3, U3.VOUT; no longer C3.1, C4.1, R3.2, R4.2, U$1.3V3, U$3.VIN
- net AIN: now also U2.IO32; no longer U$1.IO32
- net CAN_RX: no longer U$1.IO25
- net CAN_TX: no longer U$1.IO26
- net EN: now also C1.1, U$1.D1, U2.EN; no longer C1.2, U$1.EN
- net GND: now also C1.2, C3.1, C5.1, U$2.-, U2.GND, U3.GND; no longer C1.1, C3.2, U$1.GND@1, U$1.GND@2, U$3.GND
- net SCL: now also U2.IO22; no longer R2.1, U$1.IO22, U$3.SCL
- net SDA: now also U2.IO21; no longer R3.1, U$1.IO21, U$3.SDA
- net VDD_5V: now also U$2.+; no longer U$1.VIN
Other:
- moved on the sheet: C1, C2, C3, C4, R2, R4
